File: kicad-pmod_7seg.kicad_pcb (KiCad board)
At the start: 2 copper layers, 33 x 77.7 mm, 33 parts, among them J1 pmod, Q1 MMBT3906, Q2 MMBT3906, Q3 MMBT3906, Q4 MMBT3906, SW1 BTN1, SW2 BTN2, U1 7447, U2 7442, U3 CA56-12CGKWA

Commit message: 1.0
Routing:
- net +3V3: track 135.2 -> 134.3 mm
Changed lines of the file:
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@@
     (effects (font (size 1.5 1.5) (thickness 0.25) bold) (justify left bottom))
   )
-  (segment (start 147.32 86.995) (end 148.9703 86.995) (width 0.5) (layer "F.Cu") (net 1))
-  (segment (start 148.9703 86.995) (end 148.9703 64.135) (width 0.5) (layer "F.Cu") (net 1))
-  (segment (start 147.32 64.135) (end 148.9703 64.135) (width 0.5) (layer "F.Cu") (net 1))
+  (segment (start 147.955 64.135) (end 147.32 64.135) (width 0.5) (layer "F.Cu") (net 1))
   (segment (start 125.857 79.629) (end 125.857 85.471) (width 0.5) (layer "F.Cu") (net 1))
   (segment (start 139.7 69.215) (end 139.7 71.755) (width 0.5) (layer "F.Cu") (net 1))
   (segment (start 139.7 71.755) (end 139.7 74.295) (width 0.5) (layer "F.Cu") (net 1))
+  (segment (start 149.352 85.598) (end 149.352 65.532) (width 0.5) (layer "F.Cu") (net 1))
   (segment (start 127 48.26) (end 127 50.8) (width 0.5) (layer "F.Cu") (net 1))
+  (segment (start 147.955 86.995) (end 149.352 85.598) (width 0.5) (layer "F.Cu") (net 1))
+  (segment (start 147.32 86.995) (end 147.955 86.995) (width 0.5) (layer "F.Cu") (net 1))
+  (segment (start 149.352 65.532) (end 147.955 64.135) (width 0.5) (layer "F.Cu") (net 1))
   (via (at 125.857 79.629) (size 0.8) (drill 0.4) (layers "F.Cu" "B.Cu") (net 1))
   (via (at 125.857 85.471) (size 0.8) (drill 0.4) (layers "F.Cu" "B.Cu") (net 1))
@@
   (segment (start 143.2825 92.2278) (end 143.2825 92.9905) (width 0.5) (layer "B.Cu") (net 2))
   (segment (start 140.335 109.165) (end 140.335 105.41) (width 0.5) (layer "B.Cu") (net 2))
-  (segment (start 139.7 79.375) (end 141.2253 79.375) (width 0.25) (layer "F.Cu") (net 3))
   (segment (start 138.8471 60.8059) (end 138.8471 52.8282) (width 0.25) (layer "F.Cu") (net 3))
-  (segment (start 141.2253 63.1841) (end 138.8471 60.8059) (width 0.25) (layer "F.Cu") (net 3))
-  (segment (start 141.2253 79.375) (end 141.2253 63.1841) (width 0.25) (layer "F.Cu") (net 3))
-  (segment (start 139.7 50.8) (end 139.7 51.9753) (width 0.25) (layer "F.Cu") (net 3))
+  (segment (start 141.859 63.8178) (end 138.8471 60.8059) (width 0.25) (layer "F.Cu") (net 3))
   (segment (start 138.8471 52.8282) (end 139.7 51.9753) (width 0.25) (layer "F.Cu") (net 3))
-  (segment (start 148.8453 89.535) (end 148.8453 55.5004) (width 0.25) (layer "B.Cu") (net 4))
-  (segment (start 148.8453 55.5004) (end 141.6049 48.26) (width 0.25) (layer "B.Cu") (net 4))
-  (segment (start 147.32 89.535) (end 148.8453 89.535) (width 0.25) (layer "B.Cu") (net 4))
+  (segment (start 139.7 79.375) (end 140.335 79.375) (width 0.25) (layer "F.Cu") (net 3))
+  (segment (start 139.7 51.9753) (end 139.7 50.8) (width 0.25) (layer "F.Cu") (net 3))
+  (segment (start 140.335 79.375) (end 141.859 77.851) (width 0.25) (layer "F.Cu") (net 3))
+  (segment (start 141.859 77.851) (end 141.859 63.8178) (width 0.25) (layer "F.Cu") (net 3))
+  (segment (start 147.32 89.535) (end 147.701 89.535) (width 0.25) (layer "B.Cu") (net 4))
+  (segment (start 147.701 89.535) (end 149.225 88.011) (width 0.25) (layer "B.Cu") (net 4))
   (segment (start 141.6049 48.26) (end 139.7 48.26) (width 0.25) (layer "B.Cu") (net 4))
+  (segment (start 149.225 88.011) (end 149.225 55.8801) (width 0.25) (layer "B.Cu") (net 4))
+  (segment (start 149.225 55.8801) (end 141.6049 48.26) (width 0.25) (layer "B.Cu") (net 4))
   (segment (start 138.176 51.816) (end 138.176 61.119598) (width 0.25) (layer "F.Cu") (net 5))
   (segment (start 139.7 62.643598) (end 139.7 64.135) (width 0.25) (layer "F.Cu") (net 5))
   (segment (start 137.16 50.8) (end 138.176 51.816) (width 0.25) (layer "F.Cu") (net 5))
   (segment (start 138.176 61.119598) (end 139.7 62.643598) (width 0.25) (layer "F.Cu") (net 5))
+  (segment (start 138.3353 48.6274) (end 138.3353 48.26) (width 0.25) (layer "F.Cu") (net 6))
   (segment (start 148.031 54.6901) (end 142.7762 49.4353) (width 0.25) (layer "F.Cu") (net 6))
   (segment (start 139.1432 49.4353) (end 138.3353 48.6274) (width 0.25) (layer "F.Cu") (net 6))
+  (segment (start 145.415 63.627) (end 148.031 61.011) (width 0.25) (layer "F.Cu") (net 6))
+  (segment (start 145.415 90.805) (end 145.415 63.627) (width 0.25) (layer "F.Cu") (net 6))
+  (segment (start 146.685 92.075) (end 145.415 90.805) (width 0.25) (layer "F.Cu") (net 6))
+  (segment (start 138.3353 48.26) (end 137.16 48.26) (width 0.25) (layer "F.Cu") (net 6))
+  (segment (start 147.32 92.075) (end 146.685 92.075) (width 0.25) (layer "F.Cu") (net 6))
   (segment (start 142.7762 49.4353) (end 139.1432 49.4353) (width 0.25) (layer "F.Cu") (net 6))
-  (segment (start 137.16 48.26) (end 138.3353 48.26) (width 0.25) (layer "F.Cu") (net 6))
-  (segment (start 147.32 92.075) (end 145.7947 92.075) (width 0.25) (layer "F.Cu") (net 6))
-  (segment (start 145.7947 92.075) (end 145.7947 63.6334) (width 0.25) (layer "F.Cu") (net 6))
-  (segment (start 148.031 61.3971) (end 148.031 54.6901) (width 0.25) (layer "F.Cu") (net 6))
-  (segment (start 145.7947 63.6334) (end 148.031 61.3971) (width 0.25) (layer "F.Cu") (net 6))
-  (segment (start 138.3353 48.6274) (end 138.3353 48.26) (width 0.25) (layer "F.Cu") (net 6))
+  (segment (start 148.031 61.011) (end 148.031 54.6901) (width 0.25) (layer "F.Cu") (net 6))
   (segment (start 137.414 54.7693) (end 134.62 51.9753) (width 0.25) (layer "F.Cu") (net 7))
   (segment (start 138.1747 66.675) (end 137.414 65.9143) (width 0.25) (layer "F.Cu") (net 7))
@@
   (segment (start 126.6347 49.4355) (end 127.4887 49.4355) (width 0.25) (layer "B.Cu") (net 8))
   (segment (start 133.4447 47.8926) (end 133.4447 48.26) (width 0.25) (layer "B.Cu") (net 8))
+  (segment (start 139.7 76.835) (end 137.795 74.93) (width 0.25) (layer "F.Cu") (net 9))
+  (segment (start 137.795 74.93) (end 137.795 67.437) (width 0.25) (layer "F.Cu") (net 9))
   (segment (start 136.652 66.294) (end 136.652 55.372) (width 0.25) (layer "F.Cu") (net 9))
+  (segment (start 137.795 67.437) (end 136.652 66.294) (width 0.25) (layer "F.Cu") (net 9))
   (segment (start 136.652 55.372) (end 132.08 50.8) (width 0.25) (layer "F.Cu") (net 9))
-  (segment (start 139.7 76.835) (end 138.175 75.31) (width 0.25) (layer "F.Cu") (net 9))
-  (segment (start 138.175 75.31) (end 138.175 67.817) (width 0.25) (layer "F.Cu") (net 9))
-  (segment (start 138.175 67.817) (end 136.652 66.294) (width 0.25) (layer "F.Cu") (net 9))
   (segment (start 130.0968 49.4353) (end 130.9047 48.6274) (width 0.25) (layer "B.Cu") (net 10))
   (segment (start 129.2037 49.4353) (end 130.0968 49.4353) (width 0.25) (layer "B.Cu") (net 10))
@@
   (segment (start 140.6138 80.5004) (end 139.123 80.5004) (width 0.25) (layer "B.Cu") (net 27))
   (segment (start 145.0575 79.375) (end 147.32 79.375) (width 0.25) (layer "B.Cu") (net 28))
+  (segment (start 142.367 91.567) (end 140.7336 93.2004) (width 0.25) (layer "F.Cu") (net 29))
+  (segment (start 142.367 84.201) (end 142.367 91.567) (width 0.25) (layer "F.Cu") (net 29))
+  (segment (start 138.7257 93.2004) (end 136.3303 90.805) (width 0.25) (layer "F.Cu") (net 29))
   (segment (start 136.3303 90.805) (end 135.255 90.805) (width 0.25) (layer "F.Cu") (net 29))
-  (segment (start 138.7257 93.2004) (end 136.3303 90.805) (width 0.25) (layer "F.Cu") (net 29))
-  (segment (start 141.9884 91.9456) (end 140.7336 93.2004) (width 0.25) (layer "F.Cu") (net 29))
-  (segment (start 141.9884 83.8224) (end 141.9884 91.9456) (width 0.25) (layer "F.Cu") (net 29))
+  (segment (start 141.9884 83.8224) (end 142.367 84.201) (width 0.25) (layer "F.Cu") (net 29))
   (segment (start 140.7336 93.2004) (end 138.7257 93.2004) (width 0.25) (layer "F.Cu") (net 29))
   (via (at 141.9884 83.8224) (size 0.8) (drill 0.4) (layers "F.Cu" "B.Cu") (net 29))
@@
   (segment (start 132.08 86.6309) (end 134.9841 89.535) (width 0.25) (layer "B.Cu") (net 36))
   (segment (start 136.576 77.899) (end 135.7067 77.0297) (width 0.25) (layer "F.Cu") (net 37))
-  (segment (start 141.2254 90.5496) (end 141.2254 85.4982) (width 0.25) (layer "F.Cu") (net 37))
-  (segment (start 141.2254 85.4982) (end 136.576 80.8488) (width 0.25) (layer "F.Cu") (net 37))
-  (segment (start 136.576 80.8488) (end 136.576 77.899) (width 0.25) (layer "F.Cu") (net 37))
-  (segment (start 139.7 92.075) (end 141.2254 90.5496) (width 0.25) (layer "F.Cu") (net 37))
   (segment (start 130.5782 77.0297) (end 130.2882 77.3197) (width 0.25) (layer "F.Cu") (net 37))
   (segment (start 135.7067 77.0297) (end 130.5782 77.0297) (width 0.25) (layer "F.Cu") (net 37))
+  (segment (start 141.605 85.8778) (end 136.576 80.8488) (width 0.25) (layer "F.Cu") (net 37))
+  (segment (start 136.576 80.8488) (end 136.576 77.899) (width 0.25) (layer "F.Cu") (net 37))
+  (segment (start 141.605 90.17) (end 141.605 85.8778) (width 0.25) (layer "F.Cu") (net 37))
+  (segment (start 139.7 92.075) (end 141.605 90.17) (width 0.25) (layer "F.Cu") (net 37))
   (via (at 130.2882 77.3197) (size 0.8) (drill 0.4) (layers "F.Cu" "B.Cu") (net 37))
   (segment (start 130.1379 77.47) (end 130.2882 77.3197) (width 0.25) (layer "B.Cu") (net 37))
